File: pcb/MT Blade/MT Blade.kicad_pcb (KiCad board)
At the start: 2 copper layers, 105.3 x 105.3 mm, 56 parts, among them J8 Conn_01x07_Socket, J9 Conn_01x08

Commit message: code
Parts:
- added G***: LOGO, MictlanTeam-Library:MT_Blade_5mm, F.Cu at (173.8, 68.6)
- moved G 0.23 mm to (150.7, 89.6)
